File: uni02_pwm_gnerator/uni02_pwm_gnerator.kicad_sch (KiCad schematic)
At the start: 0 parts

Commit message: Updated schematic
Parts:
- added C1, C2: 10n, symbol Device:C
- added C3: 1uF, symbol Device:C
- added J1: Przewód turbinki ze sterownika, symbol Connector:Conn_01x03_Pin
- added J2: Styk sterowany ze stoiska testowego, symbol Connector:Conn_01x02_Socket
- added R1, R2: 10k, symbol Device:R
- added U1: NE555D, Package_SO:SOIC-8_3.9x4.9mm_P1.27mm, symbol Timer:NE555D
Connections:
- new net: R1.2, R2.1, U1.7 (DIS)
- new net +18V: C1.1, C2.1, J1.1 (Pin_1), J2.2 (Pin_2), R2.2, U1.8 (VCC)
- new net GND: C1.2, C2.2, C3.2, J1.3 (Pin_3), U1.1 (GND)
- new net OUT: J1.2 (Pin_2), U1.3 (Q)
- new net TR: C3.1, R1.1, U1.2 (TR), U1.6 (THR)
- new net reset: J2.1 (Pin_1), U1.4 (R)
- no-connect marks 0 -> 1
Other:
- note added: "f=1,44/(R2+2*R1)*C3 48Hz = >4L/min"

Commit message: Updated footprints
Parts:
- C1, C2: footprint (none) -> Capacitor_SMD:C_0603_1608Metric
- C3: footprint (none) -> Capacitor_SMD:CP_Elec_5x5.9
- J1: footprint (none) -> EDGE_connectors:PCB_edge 3 pin
- J2: footprint (none) -> Connector_PinHeader_2.54mm:PinHeader_1x02_P2.54mm_Vertical
- R1, R2: footprint (none) -> fResistor_SMD:R_0603_1608Metric
Connections:
- net +18V renamed +15V
Other:
- note added: "Szary - GND Czarny - PWM Czerwony - VCC"
