File: uni02_pwm_gnerator/uni02_pwm_gnerator.kicad_pcb (KiCad board)
At the start: 2 copper layers, 35 x 19 mm, 8 parts, among them J1 Przewód turbinki ze sterownika, J2 Styk sterowany ze stoiska tes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, U1 NE555D

Commit message: Final adjustments
Routing:
- net +15V: track 3.00 -> 36.0 mm
- net reset: track 0.00 -> 6.98 mm
- net GND: vias 8 -> 17
Other:
- outline, holes or cut-outs redrawn
Changed lines of the file:
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@@
 		(at 30.5 77.5)
 		(property "Reference" "J1"
-			(at 4 -7 0)
+			(at 3.6 0.1 0)
 			(unlocked yes)
 			(layer "F.SilkS")
@@
 		)
 		(property "Value" "Przewód turbinki ze sterownika"
-			(at -13 -1.5 0)
+			(at -5.9 -2.9 90)
 			(unlocked yes)
 			(layer "F.Fab")
@@
 		)
 		(fp_text user "${REFERENCE}"
-			(at -13.5 0.5 0)
+			(at -4.4 0.4 0)
 			(unlocked yes)
 			(layer "F.Fab")
@@
 		)
 		(property "Value" "Styk sterowany ze stoiska testowego"
-			(at -23.5 7.775 0)
+			(at -2.8 2.1 90)
 			(layer "F.Fab")
 			(effects
@@
 		(tags "resistor")
 		(property "Reference" "R1"
-			(at 6.225 -0.4 0)
+			(at 2.4 0.1 0)
 			(layer "F.SilkS")
 			(effects
@@
 		)
 		(property "Value" "10k"
-			(at 3.825 -0.4 0)
+			(at 4.7 0 0)
 			(layer "F.Fab")
 			(effects
@@
 		(tags "resistor")
 		(property "Reference" "R2"
-			(at 5.425 0 0)
+			(at 2.525 0.2 0)
 			(layer "F.SilkS")
 			(effects
@@
 		)
 		(property "Value" "10k"
-			(at 2.825 0 0)
+			(at 5.125 0.3 0)
 			(layer "F.Fab")
 			(effects
@@
 	)
 	(gr_line
-		(start 28 69.5)
+		(start 28 70.1)
 		(end 28 65.5)
 		(stroke
@@
 	)
 	(gr_line
-		(start 28 80.5)
+		(start 28 79.9)
 		(end 28 84.5)
 		(stroke
@@
 	(gr_line
 		(start 32.5 79.5)
-		(end 32.5 80.5)
+		(end 32.5 79.9)
 		(stroke
 			(width 0.05)
@@
 	(gr_line
 		(start 32.5 70.5)
-		(end 32.5 69.5)
+		(end 32.5 70.1)
 		(stroke
 			(width 0.05)
@@
 	)
 	(gr_line
-		(start 32.5 80.5)
-		(end 28 80.5)
+		(start 32.5 79.9)
+		(end 28 79.9)
 		(stroke
 			(width 0.05)
@@
 	)
 	(gr_line
-		(start 32.5 69.5)
-		(end 28 69.5)
+		(start 32.5 70.1)
+		(end 28 70.1)
 		(stroke
 			(width 0.05)
@@
 	)
 	(segment
+		(start 59.94 76.86)
+		(end 60.6 76.2)
+		(width 0.5)
+		(layer "F.Cu")
+		(net 1)
+	)
+	(segment
+		(start 60.6 68.4)
+		(end 58.8 66.6)
+		(width 0.5)
+		(layer "F.Cu")
+		(net 1)
+	)
+	(segment
+		(start 45 66.6)
+		(end 44.8 66.8)
+		(width 0.5)
+		(layer "F.Cu")
+		(net 1)
+	)
+	(segment
+		(start 60.6 76.2)
+		(end 60.6 68.4)
+		(width 0.5)
+		(layer "F.Cu")
+		(net 1)
+	)
+	(segment
+		(start 56.5 76.86)
+		(end 59.94 76.86)
+		(width 0.5)
+		(layer "F.Cu")
+		(net 1)
+	)
+	(segment
+		(start 58.8 66.6)
+		(end 45 66.6)
+		(width 0.5)
+		(layer "F.Cu")
+		(net 1)
+	)
+	(segment
+		(start 44.8 66.8)
+		(end 44.8 71)
+		(width 0.5)
+		(layer "F.Cu")
+		(net 1)
+	)
+	(segment
 		(start 30.5 72.5)
 		(end 33.5 72.5)
@@
 	)
 	(via
+		(at 44 80.6)
+		(size 0.6)
+		(drill 0.3)
+		(layers "F.Cu" "B.Cu")
+		(free yes)
+		(net 2)
+	)
+	(via
+		(at 43.2 66.6)
+		(size 0.6)
+		(drill 0.3)
+		(layers "F.Cu" "B.Cu")
+		(free yes)
+		(net 2)
+	)
+	(via
+		(at 58.8 75.4)
+		(size 0.6)
+		(drill 0.3)
+		(layers "F.Cu" "B.Cu")
+		(free yes)
+		(net 2)
+	)
+	(via
+		(at 51.4 78)
+		(size 0.6)
+		(drill 0.3)
+		(layers "F.Cu" "B.Cu")
+		(free yes)
+		(net 2)
+	)
+	(via
 		(at 61.5 83.5)
 		(size 0.6)
@@
 	)
 	(via
+		(at 58.6 70.6)
+		(size 0.6)
+		(drill 0.3)
+		(layers "F.Cu" "B.Cu")
+		(free yes)
+		(net 2)
+	)
+	(via
 		(at 61.5 66.8)
 		(size 0.6)
@@
 	(via
 		(at 29.5 81.5)
+		(size 0.6)
+		(drill 0.3)
+		(layers "F.Cu" "B.Cu")
+		(free yes)
+		(net 2)
+	)
+	(via
+		(at 41.4 80.6)
+		(size 0.6)
+		(drill 0.3)
+		(layers "F.Cu" "B.Cu")
+		(free yes)
+		(net 2)
+	)
+	(via
+		(at 54.2 78)
+		(size 0.6)
+		(drill 0.3)
+		(layers "F.Cu" "B.Cu")
+		(free yes)
+		(net 2)
+	)
+	(via
+		(at 42.6 70.4)
+		(size 0.6)
+		(drill 0.3)
+		(layers "F.Cu" "B.Cu")
+		(free yes)
+		(net 2)
+	)
+	(via
+		(at 51.4 72.6)
 		(size 0.6)
 		(drill 0.3)
@@
 		(layer "F.Cu")
 		(net 4)
+	)
+	(segment
+		(start 49.905 78.475)
+		(end 50.83 79.4)
+		(width 0.5)
+		(layer "F.Cu")
+		(net 5)
+	)
+	(segment
+		(start 50.83 79.4)
+		(end 56.5 79.4)
+		(width 0.5)
+		(layer "F.Cu")
+		(net 5)
 	)
 	(segment
@@
 		(min_thickness 0.25)
 		(filled_areas_thickness no)
-		(fill yes
+		(fill
 			(thermal_gap 0.5)
 			(thermal_bridge_width 0.5)
@@
 		(polygon
 			(pts
-				(xy 28.5 63) (xy 62.5 63) (xy 62.5 84) (xy 28.5 84) (xy 28.5 81) (xy 33 81) (xy 33 69) (xy 28.5 69)
-			)
-		)
+				(xy 28.5 65.9) (xy 62.5 65.9) (xy 62.5 84) (xy 28.5 84) (xy 28.5 80.6) (xy 33 80.6) (xy 33 69.5)
+				(xy 28.5 69.5)
+			)
+		)

Commit message: Updated PCB and sch
Parts:
- removed J2: Styk sterowany ze stoiska testowego, Connector_PinHeader_2.54mm:PinHeader_1x02_P2.54mm_Vertical
- added J3: Conn_01x01, EDGE_connectors:Connector_6.3mm, F.Cu at (60.9, 72.5)
- added J4: Conn_01x01, EDGE_connectors:Connector_6.3mm, F.Cu at (61.0, 83.0)
- added Q1: IRLML28003TRPBF, Package_TO_SOT_SMD:SOT-23-3, F.Cu at (37.6, 80.1)
- added R3: 50k, Resistor_SMD:R_0603_1608Metric, F.Cu at (55.0, 80.4)
- added R4: 50k, Resistor_SMD:R_0603_1608Metric, F.Cu at (42.6, 81.2)
Connections:
- J1 pad 2: OUT -> GND
- J1 pad 3: GND -> OUT_turbine
Routing:
- net OUT: track 25.8 -> 13.2 mm
- net reset: track 6.98 -> 15.8 mm
- net +15V: track 36.0 -> 28.3 mm
- net OUT_turbine: track 0.00 -> 7.04 mm
- net GND: vias 17 -> 18
Other:
- board size 35 x 19 mm -> 42 x 19 mm
